File: brands/public/Green Citrus/kicad/green_citrus_drow.sch (KiCad schematic (older format))
At the start: 48 parts

Commit message: Green Citrus layout
Parts:
- added C8: 330p, symbol CAPACITOR
- gave numbers to parts that had none: 48
Connections:
- net GND: now also C8.1
- net at C5.1, R7.1: now also P2.1; no longer P2.3
- net at C6.1, R8.2: now also P2.3; no longer P2.1
- net at C9.1: now also P3.1; no longer P3.3
- net at C10.2: now also P3.3; no longer P3.1
Other:
- moved on the sheet: B1, C7, D1, F1
