File: brands/public/Green Citrus/kicad/green_citrus_drow.sch (KiCad schematic (older format))
At the start: 49 parts, among them P1 1M Log, P2 1M RevLog, P3 1M RevLog, P4 1k Log, P5 100k Log, Q1 J201, Q2 J201, Q3 J201, Q4 J201, T1 100k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

Commit message: Green Citrus
Parts:
- C8: value 330p -> 100n
Changed lines of the file:
@@
 P 5550 2550
 F 0 "C8" H 5550 2680 59  0000 C CNN
-F 1 "330p" H 5550 2410 59  0000 C CNN
+F 1 "100n" H 5550 2410 59  0000 C CNN
 F 2 "" H 5550 2550 60  0000 C CNN
 F 3 "" H 5550 2550 60  0000 C CNN

Commit message: Green Citrus
Parts:
- P4: value 1k Log -> 1k RevLog
Connections:
- net GND: now also P4.1; no longer P4.3
- net at C5.1, R7.1: now also P2.3; no longer P2.1
- net at C6.1, R8.2: now also P2.1; no longer P2.3
- net at C9.1: now also P3.3; no longer P3.1
- net at C10.2: now also P3.1; no longer P3.3
- net at Q3.2 (S), R10.2, R13.1: now also P4.3; no longer P4.1
Changed lines of the file:
@@
 U 1 1 5490D788
 P 4500 3850
-F 0 "P2" H 4400 3950 59  0000 C CNN
+F 0 "P2" H 4600 3950 59  0000 C CNN
 F 1 "1M RevLog" H 4500 3725 59  0000 C CNN
 F 2 "" H 4500 3850 60  0000 C CNN
 F 3 "" H 4500 3850 60  0000 C CNN
 	1    4500 3850
-	0    1    -1   0
+	0    1    1    0
 $EndComp
 $Comp
@@
 U 1 1 5490E455
 P 5750 3850
-F 0 "P3" H 5650 3950 59  0000 C CNN
+F 0 "P3" H 5850 3950 59  0000 C CNN
 F 1 "1M RevLog" H 5750 3725 59  0000 C CNN
 F 2 "" H 5750 3850 60  0000 C CNN
 F 3 "" H 5750 3850 60  0000 C CNN
 	1    5750 3850
-	0    -1   -1   0
+	0    -1   1    0
 $EndComp
 $Comp
@@
 U 1 1 54911BD5
 P 6700 4100
-F 0 "P4" H 6600 4200 59  0000 C CNN
-F 1 "1k Log" H 6700 3975 59  0000 C CNN
+F 0 "P4" H 6550 4200 59  0000 C CNN
+F 1 "1k RevLog" H 6700 3975 59  0000 C CNN
 F 2 "" H 6700 4100 60  0000 C CNN
 F 3 "" H 6700 4100 60  0000 C CNN
 	1    6700 4100
-	0    -1   -1   0
+	0    -1   1    0
 $EndComp
 $Comp

Commit message: Green Citrus
Parts:
- P2, P3: value 1M RevLog -> 1M Log
- P4: value 1k RevLog -> 1k Lin
Changed lines of the file:
@@
 P 4500 3850
 F 0 "P2" H 4600 3950 59  0000 C CNN
-F 1 "1M RevLog" H 4500 3725 59  0000 C CNN
+F 1 "1M Log" H 4500 3725 59  0000 C CNN
 F 2 "" H 4500 3850 60  0000 C CNN
 F 3 "" H 4500 3850 60  0000 C CNN
@@
 P 5750 3850
 F 0 "P3" H 5850 3950 59  0000 C CNN
-F 1 "1M RevLog" H 5750 3725 59  0000 C CNN
+F 1 "1M Log" H 5750 3725 59  0000 C CNN
 F 2 "" H 5750 3850 60  0000 C CNN
 F 3 "" H 5750 3850 60  0000 C CNN
@@
 P 6700 4100
 F 0 "P4" H 6550 4200 59  0000 C CNN
-F 1 "1k RevLog" H 6700 3975 59  0000 C CNN
+F 1 "1k Lin" H 6700 3975 59  0000 C CNN
 F 2 "" H 6700 4100 60  0000 C CNN
 F 3 "" H 6700 4100 60  0000 C CNN
