File: brands/public/Engineer's Thumb/kicad/engineers_thumb.sch (KiCad schematic (older format))
At the start: 8 parts

Commit message: Engineer's Thumb, added LM13700 to KiCAD 'drow' lib
Parts:
- added C?: 10u, symbol capacitor-el
- added C?: 4.7n, symbol CAPACITOR
- added IC?: LM13700, symbol LM13700
- added P?: 10k Log, symbol POTENTIOMETER
- added R? (x2): 1k, symbol RESISTOR
- added R? (x2): 10k, symbol RESISTOR
- C?: value CAPACITOR -> 10n
- C?: value CAPACITOR -> 100p
- D? (x2): value LED -> Red
- IC?: value OPAMP_DUAL -> TL072
- P?: value POTENTIOMETER -> 1M Log
- R?: value RESISTOR -> 1k
- R?: value RESISTOR -> 10M
Other:
- moved on the sheet: C?, D?, IC?B, P?, R?

Commit message: Engineer's Thumb
Parts:
- added C3, C4: 1u, symbol capacitor-el
- added C6: 220u, symbol capacitor-el
- added C7: 100n, symbol CAPACITOR
- added C9: 47u, symbol capacitor-el
- added D3, D4, D5: 1n4148, symbol DIODE
- added unit 1 of IC1
- added unit 1 of IC2
- added IC3: TL072, symbol OPAMP_DUAL
- added P1, P3: 1M Lin, symbol POTENTIOMETER
- added Q1: BC327, TO92, symbol PNP
- added R10, R12, R13: 10k, symbol RESISTOR
- added R11: 220, symbol RESISTOR
- added R3, R9: 1M, symbol RESISTOR
- added R4, R6: 1k, symbol RESISTOR
- added SW1: SW_ON-OFF_SINGLE, symbol SW_ON-OFF_SINGLE
- gave numbers to parts that had none: 16
Connections:
- net labels added: IN, OUT, V+, Vref
- wire segments 0 -> 81
- no-connect marks 0 -> 3
Other:
- note added: "Attack"
- note added: "Bright"
- note added: "Ratio"
- note added: "Release"
- moved on the sheet: C1, C2, C5, C8, D1, D2, IC2B, P2, P4, R1, R14, R2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

Commit message: Engineer's Thumb schemetic, KiCAD libs cleanup, added CA3080
Parts:
- removed IC1: LM13700, symbol LM13700
- added B1: 9v, symbol BATTERY
- added D5: 1n4007, symbol DIODE
- added F1: FUSE, symbol FUSE
- added IC3: CA3080, symbol CA3080
- added R4: 220k, symbol RESISTOR
- R3: value 1M -> 10M
- renumbered C6 to C4, C4 to C5, C7 to C6, C9 to C7, C5 to C8, C8 to C9, D5 to D6, IC2 to IC1, IC3 to IC2, R7 to R10, R8 to R11, R9 to R12, R10 to R13, R11 to R14, R14 to R15, R4 to R5, R5 to R6, R12 to R7, R13 to R8, R6 to R9
Connections:
- wire segments 81 -> 77
- no-connect marks 3 -> 0
Other:
- note added: "Volume"
- moved on the sheet: C1, C2, C3, C4, C5, C6, C7, C8, C9, D1, D2, D3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

Commit message: Engineer's Thumb
Parts:
- added CN1: IN, symbol CONNECTOR3
- added CN2: OUT, symbol CONNECTOR2
- renumbered C5 to C4, C4 to C5
Connections:
- net GND: now also CN1.3, CN2.2; no longer B1.2
- net IN: no longer names the net of R1.2, R2.1
- net IN: now also CN1.1
- net OUT: no longer names the net of P4.2
- net OUT: now also CN2.1
- new net V-: B1.2, CN1.2
Other:
- moved on the sheet: B1, C1, C2, C3, C4, C5, C6, C7, C8, C9, D1, D2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

Commit message: added pnp transistor KiCAD footprint, added pcb file
Parts:
- B1: footprint (none) -> drow:socket_power_onboard
- C1, C8: footprint (none) -> drow:capacitor_5mm_film
- C2, C6: footprint (none) -> drow:capacitor_5mm_ceramic
- C3, C4, C7: footprint (none) -> drow:capacitor_2.5mm_electrolytic_5mm
- C5: footprint (none) -> drow:capacitor_3.5mm_electrolytic_8mm
- C9: footprint (none) -> drow:capacitor_2.5mm_tantal
- CN1, CN2: footprint (none) -> drow:socket_jack-6.35_onboard
- D1, D2: footprint (none) -> drow:diode_light_2.5mm
- D3, D4, D6: footprint (none) -> drow:diode_5mm
- D5: footprint (none) -> drow:diode_7.5mm
- F1: footprint (none) -> drow:fuse_resettable_5mm
- IC1, IC2: footprint (none) -> drow:opamp_dip8_2.5mm
- IC3: footprint (none) -> drow:ic_dip8_2.5mm
- P1, P2, P3, P4: footprint (none) -> drow:potentiometer_panel_5mm
- Q1: footprint TO92 -> drow:transistor_pnp_cbe
- R1, R10, R11, R12, R13, R14, R15, R2, R3, R4, R5, R6, R7, R8, R9: footprint (none) -> drow:resistor_7.5mm
- SW1: footprint (none) -> drow:socket_2pin_2.5mm

Commit message: Engineer's Thumb
Parts:
- CN1: footprint drow:socket_jack-6.35_onboard -> drow:socket_jack_powered-6.35_onboard
Connections:
- net GND: now also CN1.2; no longer CN1.3
- net V-: now also CN1.3; no longer CN1.2
Changed lines of the file:
@@
 $EndComp
 $Comp
-L GND #PWR2
+L GND #PWR01
 U 1 1 544D6DA5
 P 1700 4800
-F 0 "#PWR2" H 1700 4900 30  0001 C CNN
+F 0 "#PWR01" H 1700 4900 30  0001 C CNN
 F 1 "GND" H 1700 4650 30  0001 C CNN
 F 2 "" H 1700 4800 60  0000 C CNN
@@
 $EndComp
 $Comp
-L GND #PWR3
+L GND #PWR02
 U 1 1 544D6DBB
 P 2350 4800
-F 0 "#PWR3" H 2350 4900 30  0001 C CNN
+F 0 "#PWR02" H 2350 4900 30  0001 C CNN
 F 1 "GND" H 2350 4650 30  0001 C CNN
 F 2 "" H 2350 4800 60  0000 C CNN
@@
 $EndComp
 $Comp
-L GND #PWR4
+L GND #PWR03
 U 1 1 544D6DCA
 P 2650 4800
-F 0 "#PWR4" H 2650 4900 30  0001 C CNN
+F 0 "#PWR03" H 2650 4900 30  0001 C CNN
 F 1 "GND" H 2650 4650 30  0001 C CNN
 F 2 "" H 2650 4800 60  0000 C CNN
@@
 $EndComp
 $Comp
-L GND #PWR7
+L GND #PWR04
 U 1 1 544E98E3
 P 3700 4450
-F 0 "#PWR7" H 3700 4550 30  0001 C CNN
+F 0 "#PWR04" H 3700 4550 30  0001 C CNN
 F 1 "GND" H 3700 4300 30  0001 C CNN
 F 2 "" H 3700 4450 60  0000 C CNN
@@
 $EndComp
 $Comp
-L Vref #PWR21
+L Vref #PWR05
 U 1 1 544EF611
 P 7300 3400
-F 0 "#PWR21" H 7300 3370 20  0001 C CNN
+F 0 "#PWR05" H 7300 3370 20  0001 C CNN
 F 1 "Vref" H 7300 3540 59  0000 C CNN
 F 2 "" H 7300 3400 60  0000 C CNN
@@
 $EndComp
 $Comp
-L Vref #PWR24
+L Vref #PWR06
 U 1 1 544EF633
 P 8000 3800
-F 0 "#PWR24" H 8000 3770 20  0001 C CNN
+F 0 "#PWR06" H 8000 3770 20  0001 C CNN
 F 1 "Vref" H 8000 3940 59  0000 C CNN
 F 2 "" H 8000 3800 60  0000 C CNN
@@
 $EndComp
 $Comp
-L Vref #PWR5
+L Vref #PWR07
 U 1 1 544F1696
 P 3150 4800
-F 0 "#PWR5" H 3150 4770 20  0001 C CNN
+F 0 "#PWR07" H 3150 4770 20  0001 C CNN
 F 1 "Vref" H 3150 4940 59  0000 C CNN
 F 2 "" H 3150 4800 60  0000 C CNN
@@
 $EndComp
 $Comp
-L Vref #PWR22
+L Vref #PWR08
 U 1 1 544F25C4
 P 7550 2700
-F 0 "#PWR22" H 7550 2670 20  0001 C CNN
+F 0 "#PWR08" H 7550 2670 20  0001 C CNN
 F 1 "Vref" H 7550 2840 59  0000 C CNN
 F 2 "" H 7550 2700 60  0000 C CNN
@@
 $EndComp
 $Comp
-L Vref #PWR25
+L Vref #PWR09
 U 1 1 544F25E3
 P 8850 3000
-F 0 "#PWR25" H 8850 2970 20  0001 C CNN
+F 0 "#PWR09" H 8850 2970 20  0001 C CNN
 F 1 "Vref" H 8850 3140 59  0000 C CNN
 F 2 "" H 8850 3000 60  0000 C CNN
@@
 $EndComp
 $Comp
-L GND #PWR8
+L GND #PWR010
 U 1 1 544F4EFC
 P 5050 2350
-F 0 "#PWR8" H 5050 2450 30  0001 C CNN
+F 0 "#PWR010" H 5050 2450 30  0001 C CNN
 F 1 "GND" H 5050 2200 30  0001 C CNN
 F 2 "" H 5050 2350 60  0000 C CNN
@@
 $EndComp
 $Comp
-L GND #PWR10
+L GND #PWR011
 U 1 1 544F5A19
 P 5550 2350
-F 0 "#PWR10" H 5550 2450 30  0001 C CNN
+F 0 "#PWR011" H 5550 2450 30  0001 C CNN
 F 1 "GND" H 5550 2200 30  0001 C CNN
 F 2 "" H 5550 2350 60  0000 C CNN
@@
 $EndComp
 $Comp
-L GND #PWR13
+L GND #PWR012
 U 1 1 544F719F
 P 5900 2100
-F 0 "#PWR13" H 5900 2200 30  0001 C CNN
+F 0 "#PWR012" H 5900 2200 30  0001 C CNN
 F 1 "GND" H 5900 1950 30  0001 C CNN
 F 2 "" H 5900 2100 60  0000 C CNN
@@
 $EndComp
 $Comp
-L V+ #PWR6
+L V+ #PWR013
 U 1 1 544F7617
 P 3700 3950
-F 0 "#PWR6" H 3700 3920 20  0001 C CNN
+F 0 "#PWR013" H 3700 3920 20  0001 C CNN
 F 1 "V+" H 3700 4080 59  0000 C CNN
 F 2 "" H 3700 3950 60  0000 C CNN
@@
 $EndComp
 $Comp
-L V+ #PWR12
+L V+ #PWR014
 U 1 1 544F7B44
 P 5900 1600
-F 0 "#PWR12" H 5900 1570 20  0001 C CNN
+F 0 "#PWR014" H 5900 1570 20  0001 C CNN
 F 1 "V+" H 5900 1730 59  0000 C CNN
 F 2 "" H 5900 1600 60  0000 C CNN
@@
 $EndComp
 $Comp
-L V+ #PWR15
+L V+ #PWR015
 U 1 1 5450F96C
 P 6400 4750
-F 0 "#PWR15" H 6400 4720 20  0001 C CNN
+F 0 "#PWR015" H 6400 4720 20  0001 C CNN
 F 1 "V+" H 6400 4880 59  0000 C CNN
 F 2 "" H 6400 4750 60  0000 C CNN
@@
 $EndComp
 $Comp
-L GND #PWR11
+L GND #PWR016
 U 1 1 54511D5E
 P 5600 5250
-F 0 "#PWR11" H 5600 5350 30  0001 C CNN
+F 0 "#PWR016" H 5600 5350 30  0001 C CNN
 F 1 "GND" H 5600 5100 30  0001 C CNN
 F 2 "" H 5600 5250 60  0000 C CNN
@@
 $EndComp
 $Comp
-L GND #PWR14
+L GND #PWR017
 U 1 1 5451383B
 P 6000 5250
-F 0 "#PWR14" H 6000 5350 30  0001 C CNN
+F 0 "#PWR017" H 6000 5350 30  0001 C CNN
 F 1 "GND" H 6000 5100 30  0001 C CNN
 F 2 "" H 6000 5250 60  0000 C CNN
@@
 $EndComp
 $Comp
-L GND #PWR16
+L GND #PWR018
 U 1 1 5451386D
 P 6400 5800
-F 0 "#PWR16" H 6400 5900 30  0001 C CNN
+F 0 "#PWR018" H 6400 5900 30  0001 C CNN
 F 1 "GND" H 6400 5650 30  0001 C CNN
 F 2 "" H 6400 5800 60  0000 C CNN
@@
 $EndComp
 $Comp
-L GND #PWR17
+L GND #PWR019
 U 1 1 5451389F
 P 6750 5800
-F 0 "#PWR17" H 6750 5900 30  0001 C CNN
+F 0 "#PWR019" H 6750 5900 30  0001 C CNN
 F 1 "GND" H 6750 5650 30  0001 C CNN
 F 2 "" H 6750 5800 60  0000 C CNN
@@
 	6000 4850 6000 4950
 $Comp
-L PWR_FLAG #FLG1
+L PWR_FLAG #FLG020
 U 1 1 545145D7
 P 5600 4800
-F 0 "#FLG1" H 5600 4895 30  0001 C CNN
+F 0 "#FLG020" H 5600 4895 30  0001 C CNN
 F 1 "PWR_FLAG" H 5600 4980 30  0000 C CNN
 F 2 "" H 5600 4800 60  0000 C CNN
@@
 	5600 4800 5600 4950
 $Comp
-L Vref #PWR23
+L Vref #PWR021
 U 1 1 54515D4E
 P 7850 5250
-F 0 "#PWR23" H 7850 5220 20  0001 C CNN
+F 0 "#PWR021" H 7850 5220 20  0001 C CNN
 F 1 "Vref" H 7850 5390 59  0000 C CNN
 F 2 "" H 7850 5250 60  0000 C CNN
@@
 	6950 5150 6850 5150
 $Comp
-L GND #PWR20
+L GND #PWR022
 U 1 1 54519211
 P 7250 3100
-F 0 "#PWR20" H 7250 3200 30  0001 C CNN
+F 0 "#PWR022" H 7250 3200 30  0001 C CNN
 F 1 "GND" H 7250 2950 30  0001 C CNN
 F 2 "" H 7250 3100 60  0000 C CNN
@@
 $EndComp
 $Comp
-L V+ #PWR19
+L V+ #PWR023
 U 1 1 54519244
 P 7250 2600
-F 0 "#PWR19" H 7250 2570 20  0001 C CNN
+F 0 "#PWR023" H 7250 2570 20  0001 C CNN
 F 1 "V+" H 7250 2730 59  0000 C CNN
 F 2 "" H 7250 2600 60  0000 C CNN
@@
 	5050 1850 5050 2050
 $Comp
-L Vref #PWR18
+L Vref #PWR024
 U 1 1 5466C40E
 P 6900 750
-F 0 "#PWR18" H 6900 720 20  0001 C CNN
+F 0 "#PWR024" H 6900 720 20  0001 C CNN
 F 1 "Vref" H 6900 890 59  0000 C CNN
 F 2 "" H 6900 750 60  0000 C CNN
@@
 $EndComp
 $Comp
-L GND #PWR9
+L GND #PWR025
 U 1 1 546722DB
 P 5200 5250
-F 0 "#PWR9" H 5200 5350 30  0001 C CNN
+F 0 "#PWR025" H 5200 5350 30  0001 C CNN
 F 1 "GND" H 5200 5100 30  0001 C CNN
 F 2 "" H 5200 5250 60  0000 C CNN
@@
 $EndComp
 $Comp
-L GND #PWR27
+L GND #PWR026
 U 1 1 5468073B
 P 10000 4950
-F 0 "#PWR27" H 10000 5050 30  0001 C CNN
+F 0 "#PWR026" H 10000 5050 30  0001 C CNN
 F 1 "GND" H 10000 4800 30  0001 C CNN
 F 2 "" H 10000 4950 60  0000 C CNN
@@
 $EndComp
 $Comp
-L GND #PWR26
+L GND #PWR027
 U 1 1 54680773
 P 9450 4950
-F 0 "#PWR26" H 9450 5050 30  0001 C CNN
+F 0 "#PWR027" H 9450 5050 30  0001 C CNN
 F 1 "GND" H 9450 4800 30  0001 C CNN
 F 2 "" H 9450 4950 60  0000 C CNN
@@
 Text Label 4600 5350 3    60   ~ 12
 V-
-Text Label 1350 4500 0    60   ~ 12
+Text Label 1250 4900 3    60   ~ 12
 V-
 $Comp
@@
 F 0 "CN1" H 1025 4175 60  0000 C CNN
 F 1 "IN" H 1025 4875 98  0000 C CNB
-F 2 "drow:socket_jack-6.35_onboard" H 1000 4600 60  0001 C CNN
+F 2 "drow:socket_jack_powered-6.35_onboard" H 1000 4600 60  0001 C CNN
 F 3 "" H 1000 4600 60  0000 C CNN
 	1    1050 4500
@@
 	1200 4300 1850 4300
 $Comp
-L GND #PWR1
+L GND #PWR028
 U 1 1 54684A13
-P 1350 4800
-F 0 "#PWR1" H 1350 4900 30  0001 C CNN
-F 1 "GND" H 1350 4650 30  0001 C CNN
-F 2 "" H 1350 4800 60  0000 C CNN
-F 3 "" H 1350 4800 60  0000 C CNN
-	1    1350 4800
-	1    0    0    -1
-$EndComp
-Wire Wire Line
-	1350 4500 1200 4500
-Wire Wire Line
-	1200 4700 1350 4700
-Wire Wire Line
-	1350 4700 1350 4800
+P 1400 4800
+F 0 "#PWR028" H 1400 4900 30  0001 C CNN
+F 1 "GND" H 1400 4650 30  0001 C CNN
+F 2 "" H 1400 4800 60  0000 C CNN
+F 3 "" H 1400 4800 60  0000 C CNN
+	1    1400 4800
+	1    0    0    -1
+$EndComp
+Wire Wire Line
+	1200 4500 1400 4500
+Wire Wire Line
+	1400 4500 1400 4800
+Wire Wire Line
+	1200 4700 1250 4700
+Wire Wire Line
+	1250 4700 1250 4900
 $EndSCHEMATC

Commit message: Engineer's Thumb, added 3PDT switch to KiCAD lib
Parts:
- removed R3: 10M, drow:resistor_7.5mm, symbol RESISTOR
- added D6: Red, drow:diode_light_2.5mm, symbol LED
- added P1: 1M Lin, drow:potentiometer_panel_5mm, symbol POTENTIOMETER
- added R6: 10k, drow:resistor_7.5mm, symbol RESISTOR
- added SW1: SW_3PDT, drow:switch_3pdt_stomp_onboard, symbol SW_3PDT
- C3, C7: symbol capacitor-el -> CAPACITOR-EL
- C4: renamed from C5; symbol capacitor-el -> CAPACITOR-EL
- C5: renamed from C4; symbol capacitor-el -> CAPACITOR-EL
- renumbered D6 to D7, IC2 to IC1, IC1 to IC2, P1 to P2, P2 to P3, P3 to P4, P4 to P5, R4 to R3, R5 to R4, R6 to R5, SW1 to SW2
Connections:
- net +9V: now also R6.1
- net GND: now also SW1.6; no longer D5.1
- net V-: now also D5.1
- net In: now reaches R1.2, R2.1
- net In: now also SW1.5, SW1.7; no longer CN1.1
- net at C2.2, P3.1, R5.1: now also IC2.2 (-); no longer IC2.6 (-)
- net at C2.1, C9.2, P3.2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: now also IC2.1; no longer IC2.7
- net at CN2.1: now also SW1.3; no longer P5.2
- net at C5.2, R4.2: now also IC1.5 (+); no longer IC1.3 (+)
- net at D7.1, Q1.2 (B): now also IC1.7; no longer IC1.1
- net at D7.2, Q1.3 (E), R9.2: now also IC1.6 (-); no longer IC1.2 (-)
- new net: C1.2, IC2.3 (+), P1.3
- new net: IC1.3 (+), P1.2
- new net: CN1.1, SW1.9
- new net: SW1.2, SW1.8
- new net: D6.1, R6.2
- new net Led: D6.2, SW1.4
- new net Out: P5.2, SW1.1
Other:
- note added: "Threshold"
- moved on the sheet: B1, C1, C4, C6, CN1, CN2, D1, D2, D5, F1, R1, R2

Commit message: Engineer's Thumb
Connections:
- net at IC3.5, Q1.1 (C): now also R12.2; no longer R12.1
- net at R9.1: no longer R12.2
Other:
- moved on the sheet: R12
Changed lines of the file:
@@
 L RESISTOR R12
 U 1 1 544F9523
-P 7250 1500
-F 0 "R12" H 7250 1580 59  0000 C CNN
-F 1 "1M" H 7250 1400 59  0000 C CNN
-F 2 "drow:resistor_7.5mm" H 7100 1540 60  0001 C CNN
-F 3 "" H 7100 1540 60  0000 C CNN
-	1    7250 1500
+P 6450 2550
+F 0 "R12" H 6450 2630 59  0000 C CNN
+F 1 "1M" H 6450 2450 59  0000 C CNN
+F 2 "drow:resistor_7.5mm" H 6300 2590 60  0001 C CNN
+F 3 "" H 6300 2590 60  0000 C CNN
+	1    6450 2550
 	0    -1   -1   0
 $EndComp
@@
 	6450 1450 6450 1350
 Wire Wire Line
-	7250 2250 6900 2250
-Wire Wire Line
 	6900 2100 6900 2600
 Wire Wire Line
@@
 	1    0    0    -1
 $EndComp
-Connection ~ 6900 800
 Wire Wire Line
 	6900 750  6900 850
-Wire Wire Line
-	7250 800  6900 800
-Wire Wire Line
-	7250 1300 7250 800
-Wire Wire Line
-	7250 1700 7250 2250
 Wire Wire Line
 	6900 1250 6900 1600
@@
 Wire Wire Line
 	4800 5250 4800 5350
+Wire Wire Line
+	6900 2250 6450 2250
+Wire Wire Line
+	6450 2250 6450 2350
+$Comp
+L Vref #PWR?
+U 1 1 54B3E7A5
+P 6450 2750
+F 0 "#PWR?" H 6450 2720 20  0001 C CNN
+F 1 "Vref" H 6450 2890 59  0000 C CNN
+F 2 "" H 6450 2750 60  0000 C CNN
+F 3 "" H 6450 2750 60  0000 C CNN
+	1    6450 2750
+	-1   0    0    1
+$EndComp
 $EndSCHEMATC
