File: blend/fx_blender/kicad/fx_blender.sch (KiCad schematic (older format))
At the start: 54 parts, among them CN1 In, CN2 FX Send, CN3 FX Return, CN4 Out, IC1 TL072, IC2 TL072, P1 50k Lin, P2 50k Lin, P3 10k Lin, P4 100k Lin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

Commit message: FX Blender Mini
Parts:
- removed C16: 1u, ~, symbol CAPACITOR
- added C16: 10u, ~, symbol CAPACITOR-EL
- R20: value 100k -> 10k
- gave numbers to parts that had none: 2
Connections:
- net labels added: Vref
- net labels removed: VREF
- wire segments 126 -> 92
Other:
- note added: "FX Blender"
- moved on the sheet: B1, C1, C17, C2, D1, F1, R1, R2
